File: Fonte/Fonte kicad/Fonte.kicad_pcb (KiCad board)
At the start: 2 copper layers, 12 parts, among them J1 Screw_Terminal_01x03, Q1 BC547

Commit message: Add files via upload
Parts:
- added C6: 10u, Capacitor_THT:CP_Radial_D10.0mm_P7.50mm, F.Cu at (287.1, 27.9)
- added C7: 100n, Capacitor_THT:CP_Radial_D10.0mm_P7.50mm, F.Cu at (226.4, 73.5)
- added D10: LED, LED_THT:LED_D5.0mm, F.Cu at (172.8, 30.5)
- added D11: LED, LED_THT:LED_D5.0mm, F.Cu at (180.3, 30.5)
- added D12: LED, LED_THT:LED_D5.0mm, F.Cu at (158.4, 28.7)
- added D6: 1N53xxB, Diode_THT:D_DO-41_SOD81_P10.16mm_Horizontal, F.Cu at (212.1, 69.8)
- added D7: 1N4007, Diode_THT:D_DO-41_SOD81_P10.16mm_Horizontal, F.Cu at (212.1, 74.1)
- added D8: 1N4007, Diode_THT:D_DO-41_SOD81_P10.16mm_Horizontal, F.Cu at (212.1, 78.3)
- added D9: 1N53xxB, Diode_THT:D_DO-41_SOD81_P10.16mm_Horizontal, F.Cu at (212.1, 82.6)
- added HS1: Heatsink, Heatsink:Heatsink_Stonecold_HS-132_32x14mm_2xFixation1.5mm, F.Cu at (130.8, 2.54)
- added J2: Conn_02x02_Top_Bottom, Package_DIP:DIP-4_W10.16mm, F.Cu at (111.1, 43.2)
- added J3: Screw_Terminal_01x02, TerminalBlock_Phoenix:TerminalBlock_Phoenix_MKDS-1,5-2_1x02_P5.00mm_Horizontal, F.Cu at (238.8, -2.54)
- added J4: Screw_Terminal_01x02, TerminalBlock_Phoenix:TerminalBlock_Phoenix_MKDS-1,5-2_1x02_P5.00mm_Horizontal, F.Cu at (276.3, 28.4)
- added JP2: Jumper_2_Bridged, TestPoint:TestPoint_2Pads_Pitch2.54mm_Drill0.8mm, F.Cu at (225.9, 86.9)
- added K2: Relay_SPDT, Relay_THT:Relay_SPDT_Finder_40.31, F.Cu at (80.0, 14.1)
- added Q2: BC556, Package_TO_SOT_THT:TO-92_Inline, F.Cu at (205.7, 70.9)
- added Q3: BC556, Package_TO_SOT_THT:TO-92_Inline, F.Cu at (205.7, 76.7)
- added Q4: IRF540N, Package_TO_SOT_THT:TO-220-3_Vertical, F.Cu at (128.3, 4.12)
- added Q5: 2N7000, Package_TO_SOT_THT:TO-92_Inline, F.Cu at (205.7, 82.5)
- added Q6: BC547, Package_TO_SOT_THT:TO-92_Inline, F.Cu at (205.7, 88.3)
- added R10: R, Resistor_THT:R_Axial_DIN0207_L6.3mm_D2.5mm_P10.16mm_Horizontal, F.Cu at (175.3, 73.2)
- added R10: R, Resistor_THT:R_Axial_DIN0207_L6.3mm_D2.5mm_P10.16mm_Horizontal, F.Cu at (192.0, 61.8)
- added R11: R, Resistor_THT:R_Axial_DIN0207_L6.3mm_D2.5mm_P10.16mm_Horizontal, F.Cu at (157.5, 22.9)
- added R12: R, Resistor_THT:R_Axial_DIN0207_L6.3mm_D2.5mm_P10.16mm_Horizontal, F.Cu at (175.3, 77.2)
- added R13: R, Resistor_THT:R_Axial_DIN0207_L6.3mm_D2.5mm_P10.16mm_Horizontal, F.Cu at (192.0, 65.8)
- added R14: R, Resistor_THT:R_Axial_DIN0207_L6.3mm_D2.5mm_P10.16mm_Horizontal, F.Cu at (192.0, 69.9)
- added R15: R, Resistor_THT:R_Axial_DIN0207_L6.3mm_D2.5mm_P10.16mm_Horizontal, F.Cu at (192.0, 73.9)
- added R16: R, Resistor_THT:R_Axial_DIN0207_L6.3mm_D2.5mm_P10.16mm_Horizontal, F.Cu at (192.0, 78.0)
- added R17: R, Resistor_THT:R_Axial_DIN0207_L6.3mm_D2.5mm_P10.16mm_Horizontal, F.Cu at (192.0, 82.0)
- added R18: R, Resistor_THT:R_Axial_DIN0207_L6.3mm_D2.5mm_P10.16mm_Horizontal, F.Cu at (192.0, 86.1)
- added R19: R, Resistor_THT:R_Axial_DIN0207_L6.3mm_D2.5mm_P10.16mm_Horizontal, F.Cu at (246.4, 40.6)
- added R2: R_Small, Diode_THT:D_P600_R-6_P20.00mm_Horizontal, F.Cu at (170.3, 0.00)
- added R20: R, Resistor_THT:R_Axial_DIN0207_L6.3mm_D2.5mm_P10.16mm_Horizontal, F.Cu at (175.3, 81.3)
- added R3: R, Resistor_THT:R_Axial_DIN0207_L6.3mm_D2.5mm_P10.16mm_Horizontal, F.Cu at (274.4, 20.1)
- added R4: R, Resistor_THT:R_Axial_DIN0207_L6.3mm_D2.5mm_P10.16mm_Horizontal, F.Cu at (124.5, 43.2)
- added R5: R, Resistor_THT:R_Axial_DIN0207_L6.3mm_D2.5mm_P10.16mm_Horizontal, F.Cu at (192.0, 41.5)
- added R6: R, Resistor_THT:R_Axial_DIN0207_L6.3mm_D2.5mm_P10.16mm_Horizontal, F.Cu at (192.0, 45.6)
- added R7: R, Resistor_THT:R_Axial_DIN0207_L6.3mm_D2.5mm_P10.16mm_Horizontal, F.Cu at (192.0, 49.6)
- added R8: R, Resistor_THT:R_Axial_DIN0207_L6.3mm_D2.5mm_P10.16mm_Horizontal, F.Cu at (192.0, 53.7)
- added R9: R, Resistor_THT:R_Axial_DIN0207_L6.3mm_D2.5mm_P10.16mm_Horizontal, F.Cu at (192.0, 57.7)
- added RV1: R_Potentiometer, Potentiometer_THT:Potentiometer_Piher_PC-16_Single_Horizontal, F.Cu at (206.0, 53.3)
- added RV2: R_Potentiometer, Potentiometer_THT:Potentiometer_Piher_PC-16_Single_Horizontal, F.Cu at (203.4, 12.6)
- added U1: LM324, Package_DIP:DIP-14_W7.62mm, F.Cu at (167.6, 43.2)
- C1: footprint Capacitor_THT:CP_Radial_D30.0mm_P10.00mm_SnapIn -> Capacitor_THT:CP_Radial_D22.0mm_P10.00mm_SnapIn
- C2, C3: footprint Capacitor_THT:CP_Axial_L18.0mm_D6.5mm_P25.00mm_Horizontal -> Capacitor_THT:CP_Radial_D12.5mm_P5.00mm
- D5: footprint Diode_THT:D_DO-201AD_P12.70mm_Horizontal -> Diode_THT:D_DO-41_SOD81_P10.16mm_Horizontal
- R1: footprint Resistor_THT:R_Axial_DIN0918_L18.0mm_D9.0mm_P7.62mm_Vertical -> Resistor_THT:R_Axial_DIN0207_L6.3mm_D2.5mm_P10.16mm_Horizontal
- moved C4 116.8 mm to (195.6, 15.4)
- moved D3 62.0 mm to (35.6, 43.2), turned to -90 degrees
- moved Q1 56.3 mm to (78.9, 43.2)
- moved R1 56.3 mm to (61.1, 43.2)
- moved C2 53.6 mm to (27.8, 48.3)
- moved C3 53.6 mm to (48.3, 43.4)
- moved D4 53.6 mm to (28.0, 53.4)
- moved D5 33.3 mm to (119.4, 78.7)
- moved D2 26.4 mm to (40.6, 30.6)
- moved C1 26.4 mm to (58.4, 20.5)
- moved D1 26.4 mm to (40.6, 20.5)
- moved J1 26.4 mm to (22.6, 20.5)
Routing:
- net Net-(D3-K): track 42.7 -> 0.00 mm
- net Net-(D10-A): track 0.00 -> 30.0 mm
- net Net-(D5-K): track 25.7 -> 0.00 mm
- net V_in: track 46.2 -> 26.3 mm
- net GND: track 108.4 -> 100.6 mm
- net VCC: track 5.20 -> 0.00 mm
- net Net-(D3-A): track 10.5 -> 12.8 mm
Other:
- board outline added: 220.2 x 99.1 mm

Commit message: Add files via upload
Parts:
- removed C4: 100n, Capacitor_THT:CP_Axial_L10.0mm_D6.0mm_P15.00mm_Horizontal
- removed JP2: Jumper_2_Bridged, TestPoint:TestPoint_2Pads_Pitch2.54mm_Drill0.8mm
- removed K2: Relay_SPDT, Relay_THT:Relay_SPDT_Finder_40.31
- removed the R10 at (175.3, 73.2)
- removed R15: R, Resistor_THT:R_Axial_DIN0207_L6.3mm_D2.5mm_P10.16mm_Horizontal
- added K1: SANYOU_SRD_Form_C, Relay_THT:Relay_SPDT_SANYOU_SRD_Series_Form_C, F.Cu at (61.6, 26.9)
- added RV3: R_Potentiometer, Potentiometer_THT:Potentiometer_Piher_PC-16_Single_Horizontal, F.Cu at (166.0, 58.4)
- added RV3: R_Potentiometer_Trim, Resistor_THT:R_Axial_DIN0204_L3.6mm_D1.6mm_P1.90mm_Vertical, F.Cu at (197.8, 61.6)
- Q1, Q2, Q3, Q5, Q6: footprint Package_TO_SOT_THT:TO-92_Inline -> Package_TO_SOT_THT:TO-92L_Wide
- R2: footprint Diode_THT:D_P600_R-6_P20.00mm_Horizontal -> Resistor_THT:R_Axial_DIN0516_L15.5mm_D5.0mm_P5.08mm_Vertical
- moved J4 253.0 mm to (24.3, 50.2), turned to -90 degrees
- moved R3 208.4 mm to (70.5, 63.5), turned to -90 degrees
- moved C6 194.5 mm to (103.5, 92.1)
- moved D9 193.9 mm to (22.1, 43.8), turned to 90 degrees
- moved R18 173.0 mm to (27.3, 33.0), turned to -90 degrees
- moved R13 171.1 mm to (21.0, 61.6), turned to -90 degrees
- moved C7 161.6 mm to (66.0, 93.5), turned to -90 degrees
- moved D8 160.5 mm to (52.7, 59.7), turned to -90 degrees
- moved D11 159.1 mm to (25.4, 66.7)
- moved R14 156.6 mm to (36.2, 54.0), turned to -90 degrees
- moved D7 155.6 mm to (59.1, 45.7), turned to -90 degrees
- moved Q6 155.1 mm to (54.6, 53.1), turned to 180 degrees
- moved RV2 151.0 mm to (81.4, 101.6), turned to -90 degrees
- moved Q5 149.6 mm to (56.3, 74.1), turned to 180 degrees
- moved D6 147.4 mm to (64.8, 64.1), turned to -90 degrees
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Connections:
- D11 pad 2: NO -> Net-(D11-A)
- D8 pad 1: Net-(D8-K) -> Net-(D11-K)
- J2 pad 1: GND -> unconnected-(J2-Pin_1-Pad1)
- J2 pad 3: Net-(D8-K) -> unconnected-(J2-Pin_3-Pad3)
- J2 pad 4: Net-(D8-K) -> Net-(D11-K)
- Q6 pad 2: Net-(D8-K) -> Net-(D11-K)
- R17 pad 2: V_ret -> Net-(K1-Pad2)
- R4 pad 1: Net-(D11-K) -> NO
- R4 pad 2: Net-(D8-K) -> Net-(D11-A)
- U1 pad 12: (no net) -> GND
- U1 pad 13: (no net) -> Net-(U1D--)
- U1 pad 14: (no net) -> Net-(U1D--)
Routing:
- net Net-(Q2-E): track 0.00 -> 77.0 mm
- net GND: track 100.6 -> 24.7 mm
- net V_in: track 26.3 -> 83.3 mm
- net Net-(D11-K): track 0.00 -> 56.4 mm
- net Net-(U1C--): track 0.00 -> 52.4 mm
- net NO: track 0.00 -> 42.5 mm
- net Net-(D7-A): track 0.00 -> 38.9 mm
- net V_ret: track 27.9 -> 65.3 mm
- net Net-(D3-K): track 0.00 -> 36.2 mm
- net Net-(J3-Pin_1): track 0.00 -> 32.8 mm
- net Net-(Q4-S): track 0.00 -> 29.1 mm
- net Net-(D9-K): track 0.00 -> 26.1 mm
- net Net-(U1A-+): track 0.00 -> 26.1 mm
- net Net-(D11-A): track 0.00 -> 22.2 mm
- net Net-(R11-Pad1): track 0.00 -> 19.8 mm
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Other:
- board size 220.2 x 99.1 mm -> 100 x 100 mm

Commit message: Add files via upload
Parts:
- removed R14: R, Resistor_THT:R_Axial_DIN0207_L6.3mm_D2.5mm_P10.16mm_Horizontal
- removed the RV3 at (166.0, 58.4)
- removed the RV3 at (197.8, 61.6)
- added RV3: R_Potentiometer, TerminalBlock_Philmore:TerminalBlock_Philmore_TB133_1x03_P5.00mm_Horizontal, F.Cu at (85.7, 84.2)
- moved R4 28.4 mm to (34.9, 57.1), turned to -90 degrees
- moved R6 11.2 mm to (95.2, 33.2), turned to 180 degrees
- moved R8 10.6 mm to (85.1, 29.4), turned to 0 degrees
- moved R10 10.3 mm to (74.9, 92.7), turned to 90 degrees
- moved U1 8.36 mm to (94.0, 61.6)
- moved J2 4.59 mm to (28.6, 75.6), turned to 0 degrees
- moved R7 4.49 mm to (99.7, 42.5)
- moved C6 3.47 mm to (104.9, 88.9)
- moved D10 3.42 mm to (45.1, 67.9), turned to 0 degrees
- moved R18 2.54 mm to (29.8, 33.0)
- moved D11 2.29 mm to (27.3, 65.4)
- moved R11 1.51 mm to (83.7, 25.4)
- moved R3 1.27 mm to (69.2, 63.5)
Routing:
- net Net-(Q5-G): track 4.53 -> 230.1 mm
- net Net-(R9-Pad2): track 0.00 -> 151.8 mm
- net Net-(D10-A): track 43.7 -> 192.7 mm
- net Net-(J4-Pin_2): track 7.77 -> 129.0 mm
- net Net-(D9-K): track 26.1 -> 121.6 mm
- net VCC: track 12.9 -> 86.0 mm
- net Net-(R16-Pad1): track 17.3 -> 85.7 mm
- net V_ref: track 9.79 -> 69.1 mm
- net NO: track 42.5 -> 94.3 mm
- net Net-(U1C--): track 52.4 -> 18.9 mm
- net Net-(U1B--): track 3.18 -> 32.6 mm
- net GND: track 24.7 -> 0.52 mm
- net Net-(U1A-+): track 26.1 -> 3.81 mm
- net Net-(R11-Pad1): track 19.8 -> 38.3 mm
- net Net-(D11-A): track 22.2 -> 6.77 mm
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
Commit message: Add files via upload
Parts:
- moved R13 0.64 mm to (21.6, 61.6)
- moved R18 0.63 mm to (29.8, 33.7)
- moved D10 0.63 mm to (45.1, 67.3)
- moved R19 0.59 mm to (109.5, 45.1)
Routing:
- net Net-(U1A-+): track 3.81 -> 28.1 mm
- net Net-(R9-Pad2): track 151.8 -> 144.2 mm
- net Net-(R16-Pad1): track 85.7 -> 79.4 mm
- net Net-(D10-A): track 192.7 -> 188.0 mm
- net Net-(Q5-G): track 230.1 -> 226.1 mm
- net V_ref: track 69.1 -> 65.6 mm
- net Net-(U1A--): track 8.19 -> 11.4 mm
- net V_ret: track 64.2 -> 61.3 mm
- net NO: track 94.3 -> 91.6 mm
- net Net-(U1D--): track 0.00 -> 2.54 mm
- net Net-(J3-Pin_1): track 35.5 -> 33.4 mm
- net VCC: track 86.0 -> 83.9 mm
- net Net-(D9-K): track 121.6 -> 120.5 mm
- net Net-(Q4-S): track 32.6 -> 31.6 mm
- net Net-(D11-A): track 6.77 -> 5.87 mm
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
Commit message: Add files via upload
Parts:
- Q4: footprint Package_TO_SOT_THT:TO-220-3_Vertical -> Package_TO_SOT_THT:TO-218-3_Vertical
- moved R13 59.4 mm to (74.4, 88.6)
- moved R8 28.6 mm to (86.9, 57.9), turned to 180 degrees
- moved R16 21.6 mm to (57.4, 81.3), turned to 90 degrees
- moved R6 14.3 mm to (92.5, 47.2), turned to -90 degrees
- moved R9 10.8 mm to (96.0, 47.2), turned to -90 degrees
- moved R20 9.61 mm to (102.9, 67.9), turned to 0 degrees
- moved R7 9.09 mm to (95.9, 34.3), turned to -90 degrees
- moved D5 8.47 mm to (58.2, 104.4), turned to 0 degrees
- moved R3 8.47 mm to (67.3, 71.8)
- moved D6 7.65 mm to (63.2, 71.6)
- moved Q5 7.24 mm to (51.8, 79.8), turned to 90 degrees
- moved R11 6.69 mm to (79.4, 30.5)
- moved R10 5.73 mm to (80.5, 94.0)
- moved Q4 5.41 mm to (86.0, 14.0)
- moved D12 4.12 mm to (111.1, 61.0), turned to 180 degrees
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Routing:
- net Net-(R9-Pad2): track 144.2 -> 55.2 mm
- net Net-(D6-K): track 6.85 -> 61.8 mm
- net Net-(R16-Pad1): track 79.4 -> 29.3 mm
- net Net-(U1A-+): track 28.1 -> 10.1 mm
- net Net-(D10-A): track 188.0 -> 205.9 mm
- net Net-(Q5-G): track 226.1 -> 209.4 mm
- net Net-(Q4-S): track 31.6 -> 43.1 mm
- net Net-(U1B--): track 32.1 -> 42.1 mm
- net Net-(U1A--): track 11.4 -> 20.5 mm
- net Net-(R11-Pad1): track 38.3 -> 31.4 mm
- net Net-(Q2-C): track 14.1 -> 20.4 mm
- net Net-(Q2-E): track 86.3 -> 81.6 mm
- net Net-(D5-K): track 16.4 -> 20.3 mm
- net Net-(J4-Pin_2): track 129.0 -> 125.7 mm
- net Net-(J3-Pin_1): track 33.4 -> 36.2 mm
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- added copper zone on B.Cu, net GND
Other:
- board text added: "J1"
- board text added: "J3"

Commit message: Add files via upload
Parts:
- moved D2 1.92 mm to (40.3, 23.5)
- moved R18 0.18 mm to (30.0, 33.5)
Routing:
- net V_in: track 83.3 -> 84.3 mm
- net NO: track 90.6 -> 91.2 mm

Commit message: Add files via upload
Parts:
- removed R10, R17: R, Resistor_THT:R_Axial_DIN0207_L6.3mm_D2.5mm_P10.16mm_Horizontal
- added R14: 100, Resistor_THT:R_Axial_DIN0207_L6.3mm_D2.5mm_P10.16mm_Horizontal, F.Cu at (59.1, 43.2)
- D1, D2: footprint Diode_THT:D_DO-41_SOD81_P10.16mm_Horizontal -> Diode_THT:D_DO-41_SOD81_P12.70mm_Horizontal
- R2: footprint Resistor_THT:R_Axial_DIN0516_L15.5mm_D5.0mm_P5.08mm_Vertical -> Resistor_THT:R_Axial_DIN0207_L6.3mm_D2.5mm_P10.16mm_Horizontal
- R6: footprint Resistor_THT:R_Axial_DIN0207_L6.3mm_D2.5mm_P10.16mm_Horizontal -> Resistor_THT:R_Axial_DIN0309_L9.0mm_D3.2mm_P12.70mm_Horizontal
- moved R11 20.9 mm to (77.5, 51.3), turned to 90 degrees
- moved R2 13.5 mm to (91.9, 29.7), turned to 0 degrees
- moved R6 6.11 mm to (88.1, 42.9)
- moved C2 5.64 mm to (24.4, 91.9)
- moved R13 5.09 mm to (74.2, 93.7)
- moved RV3 4.87 mm to (84.6, 88.9)
- moved Q1 4.69 mm to (55.9, 89.9)
- moved C3 4.59 mm to (40.6, 89.6)
- moved R12 4.24 mm to (105.9, 46.5)
- moved D4 3.87 mm to (24.4, 102.9)
- moved C7 3.68 mm to (66.0, 89.9)
- moved R8 3.10 mm to (85.1, 55.4)
- moved Q4 1.98 mm to (86.0, 15.9)
- moved D3 1.91 mm to (31.1, 89.5)
- moved D1 1.90 mm to (41.9, 15.2)
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Connections:
- net Net-(D1-A) renamed /V_in+
- net Net-(D10-A) renamed /V_Led_Lrg
- net Net-(D11-A) renamed /V_Led_Red
- net Net-(D12-A) renamed /V_Led_G
- net Net-(D5-K) renamed /V_ref_VCC
- net Net-(D9-K) renamed /V_Ref_T
- net Net-(J3-Pin_1) renamed /V_out
- net Net-(J4-Pin_2) renamed V_ntc
- net Net-(Q4-S) renamed /V_shant
- net Net-(Q5-G) renamed /V_max_A
- net Net-(R16-Pad1) renamed /V_op_T
- net Net-(R9-Pad2) renamed /V_dif_op
- net Net-(U1B--) renamed /V_Vmax-
- net Net-(U1C--) renamed /V_max_T
- net V_in renamed /V_in-
- C6 pad 1: V_ref -> /V_Vmax
- D6 pad 1: Net-(D6-K) -> V_ref
- K1 pad 2: Net-(K1-Pad2) -> Net-(D7-K)
- Q3 pad 1: Net-(D6-K) -> V_ref
- RV1 pad 1: Net-(D6-K) -> V_ref
- RV1 pad 2: V_ref -> /V_Vmax
- U1 pad 5: V_ref -> /V_Vmax
Routing:
- net /V_Led_Lrg: track 205.9 -> 90.4 mm
- net /V_Vmax: track 0.00 -> 93.1 mm
- net Net-(D6-K): track 61.8 -> 0.00 mm
- net /V_max_A: track 209.4 -> 172.1 mm
- net /V_Vmax-: track 42.1 -> 68.3 mm
- net Net-(R11-Pad1): track 31.4 -> 10.3 mm
- net Net-(D7-K): track 3.17 -> 23.0 mm
- net /V_shant: track 43.1 -> 30.6 mm
- net Net-(K1-Pad2): track 10.6 -> 0.00 mm
- net Net-(Q2-B): track 14.1 -> 4.04 mm
- net V_ret: track 62.1 -> 69.0 mm
- net /V_in-: track 84.3 -> 78.3 mm
- net Net-(Q2-E): track 81.6 -> 87.1 mm
- net Net-(D3-A): track 15.5 -> 20.4 mm
- net V_ref: track 67.8 -> 63.0 mm
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Other:
- board text removed: "J1"
