File: Fonte/Fonte kicad/Fonte.kicad_sch (KiCad schematic)
At the start: 45 parts, among them J2 Screw_Terminal_01x01, J2 Screw_Terminal_01x03, K2 Relay_SPDT, Q1 BC547, Q2 BC556, Q3 BC556, Q4 IRF540N, Q5 2N7000, Q6 BC547, U1 LM324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

Commit message: Add files via upload
Parts:
- removed J2: Screw_Terminal_01x01, symbol Connector:Screw_Terminal_01x01
- removed R10: R, symbol Device:R
- removed TH1: Thermistor_NTC, symbol Device:Thermistor_NTC
- added D10, D11, D12: LED, LED_THT:LED_D5.0mm, symbol Device:LED
- added J2: Conn_02x02_Top_Bottom, Package_DIP:DIP-4_W10.16mm, symbol Connector_Generic:Conn_02x02_Top_Bottom
- added J3, J4: Screw_Terminal_01x02, TerminalBlock_Phoenix:TerminalBlock_Phoenix_MKDS-1,5-2_1x02_P5.00mm_Horizontal, symbol Connector:Screw_Terminal_01x02
- added R12, R19, R20, R4: R, Resistor_THT:R_Axial_DIN0207_L6.3mm_D2.5mm_P10.16mm_Horizontal, symbol Device:R
- added RV2: R_Potentiometer, Potentiometer_THT:Potentiometer_Piher_PC-16_Single_Horizontal, symbol Device:R_Potentiometer
- added unit 5 of U1
- C1: footprint Capacitor_THT:CP_Radial_D30.0mm_P10.00mm_SnapIn -> Capacitor_THT:CP_Radial_D22.0mm_P10.00mm_SnapIn
- C2, C3: footprint Capacitor_THT:CP_Axial_L18.0mm_D6.5mm_P25.00mm_Horizontal -> Capacitor_THT:CP_Radial_D12.5mm_P5.00mm
- C6: value C -> 10u; footprint (none) -> Capacitor_THT:CP_Radial_D10.0mm_P7.50mm
- C7: value C -> 100n; footprint (none) -> Capacitor_THT:CP_Radial_D10.0mm_P7.50mm
- D5: footprint Diode_THT:D_DO-201AD_P12.70mm_Horizontal -> Diode_THT:D_DO-41_SOD81_P10.16mm_Horizontal
- D6, D9: footprint Diode_THT:D_DO-201_P15.24mm_Horizontal -> Diode_THT:D_DO-41_SOD81_P10.16mm_Horizontal
- HS1: footprint (none) -> Heatsink:Heatsink_Stonecold_HS-132_32x14mm_2xFixation1.5mm
- K2: footprint (none) -> Relay_THT:Relay_SPDT_Finder_40.31
- R1: footprint Resistor_THT:R_Axial_DIN0918_L18.0mm_D9.0mm_P7.62mm_Vertical -> Resistor_THT:R_Axial_DIN0207_L6.3mm_D2.5mm_P10.16mm_Horizontal
- R11, R13, R14, R15, R16, R17, R18, R3, R5, R6, R7, R8, R9: footprint (none) -> Resistor_THT:R_Axial_DIN0207_L6.3mm_D2.5mm_P10.16mm_Horizontal
- R2: footprint (none) -> Diode_THT:D_P600_R-6_P20.00mm_Horizontal
- RV1: footprint Potentiometer_SMD:Potentiometer_ACP_CA6-VSMD_Vertical -> Potentiometer_THT:Potentiometer_Piher_PC-16_Single_Horizontal
- U1: footprint (none) -> Package_DIP:DIP-14_W7.62mm
- U1: renamed from U2; footprint (none) -> Package_DIP:DIP-14_W7.62mm
- U1: renamed from U3; footprint (none) -> Package_DIP:DIP-14_W7.62mm
Connections:
- net GND: now also R13.2, R15.2, D12.1 (K), J2.1 (Pin_1), J2.2 (Pin_2), J3.2 (Pin_2), R20.2, RV2.1, U1.11 (V-); no longer R13.1, U1.10 (+)
- net VCC: now also U1.4 (V+)
- net V_ret: now also K2.A2, R17.2
- net at Q4.1 (G), R11.2: now also D10.2 (A); no longer Q5.3 (D)
- net at R9.2: now also U1.1, RV2.3; no longer U1.6 (-)
- net at D8.1 (K), Q6.2 (B): now also J2.3 (Pin_3), J2.4 (Pin_4), R4.2
- net at R2.2, R7.1: now also J3.1 (Pin_1), R12.1, R19.1
- net at D9.1 (K), R14.1, R18.2: now also J4.1 (Pin_1)
- net at Q5.2 (G): now also RV2.2; no longer U1.1
- net NO: now reaches K2.14
- net NO: now also D11.2 (A)
- new net: J4.2 (Pin_2), R13.1, U1.10 (+)
- new net: D10.1 (K), Q5.3 (D)
- new net: D12.2 (A), R19.2
- new net: R12.2, R20.1, U1.6 (-)
- new net: D11.1 (K), R4.1
Other:
- moved on the sheet: HS1, Q5, R13, R14

Commit message: Add files via upload
Parts:
- removed K2: Relay_SPDT, Relay_THT:Relay_SPDT_Finder_40.31, symbol Relay:Relay_SPDT
- removed R14, R15: R, Resistor_THT:R_Axial_DIN0207_L6.3mm_D2.5mm_P10.16mm_Horizontal, symbol Device:R
- added K1: SANYOU_SRD_Form_C, Relay_THT:Relay_SPDT_SANYOU_SRD_Series_Form_C, symbol Relay:SANYOU_SRD_Form_C
- added RV3: R_Potentiometer, Potentiometer_THT:Potentiometer_Piher_PC-16_Single_Horizontal, symbol Device:R_Potentiometer
- added unit 4 of U1
- Q1, Q2, Q3, Q5, Q6: footprint Package_TO_SOT_THT:TO-92_Inline -> Package_TO_SOT_THT:TO-92L_Wide
- R2: footprint Diode_THT:D_P600_R-6_P20.00mm_Horizontal -> Resistor_THT:R_Axial_DIN0516_L15.5mm_D5.0mm_P5.08mm_Vertical
Connections:
- net GND: now also RV3.3, U1.12 (+); no longer J2.1 (Pin_1)
- net NO: now also R4.1, K1.3; no longer D11.2 (A)
- net V_ret: now also K1.1; no longer R17.2
- net at D8.1 (K), J2.4 (Pin_4), Q6.2 (B): now also D11.1 (K); no longer J2.3 (Pin_3), R4.2
- net at Q2.3 (E), Q4.2 (D), R5.1: now also K1.4
- net at D9.1 (K), J4.1 (Pin_1), R18.2: now also RV3.1
- net at D7.2 (A), Q6.1 (C): now also K1.5
- net at U1.9 (-): now also RV3.2
- new net: K1.2, R17.2
- new net: D11.2 (A), R4.2
- new net: U1.13 (-), U1.14
Other:
- moved on the sheet: D11, D7, R17, R4

Commit message: Add files via upload
Parts:
- RV3: footprint Potentiometer_THT:Potentiometer_Piher_PC-16_Single_Horizontal -> TerminalBlock_Philmore:TerminalBlock_Philmore_TB133_1x03_P5.00mm_Horizontal
Changed lines of the file:
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@@
       (effects (font (size 1.27 1.27)) (justify right))
     )
-    (property "Footprint" "Potentiometer_THT:Potentiometer_Piher_PC-16_Single_Horizontal" (at 111.76 59.69 0)
+    (property "Footprint" "TerminalBlock_Philmore:TerminalBlock_Philmore_TB133_1x03_P5.00mm_Horizontal" (at 111.76 59.69 0)
       (effects (font (size 1.27 1.27)) hide)
     )

Commit message: Add files via upload
Parts:
- Q4: footprint Package_TO_SOT_THT:TO-220-3_Vertical -> Package_TO_SOT_THT:TO-218-3_Vertical
Changed lines of the file:
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@@
       (effects (font (size 1.27 1.27)))
     )
-    (property "Footprint" "Package_TO_SOT_THT:TO-220-3_Vertical" (at 238.125 26.67 0)
+    (property "Footprint" "Package_TO_SOT_THT:TO-218-3_Vertical" (at 238.125 26.67 0)
       (effects (font (size 1.27 1.27) italic) (justify left) hide)
     )

Commit message: Add files via upload
Parts:
- removed R17: R, Resistor_THT:R_Axial_DIN0207_L6.3mm_D2.5mm_P10.16mm_Horizontal, symbol Device:R
- added R14: 100, Resistor_THT:R_Axial_DIN0207_L6.3mm_D2.5mm_P10.16mm_Horizontal, symbol Device:R
- R2: footprint Resistor_THT:R_Axial_DIN0516_L15.5mm_D5.0mm_P5.08mm_Vertical -> Resistor_THT:R_Axial_DIN0207_L6.3mm_D2.5mm_P10.16mm_Horizontal
Connections:
- net V_ref: now also D6.1 (K), Q3.1 (C), RV1.1; no longer C6.1, RV1.2, U1.5 (+)
- net V_ret: now also R14.2
- net V_ref_VCC: now reaches D5.1 (K), Q1.2 (B), R1.2
- net V_Led_Lrg: now reaches D10.2 (A), Q4.1 (G), R11.2
- net V_dif_op: now reaches R9.2, RV2.3, U1.1
- net V_in+: now reaches D1.2 (A), J2.1 (Pin_1)
- net V_Ref_T: now reaches D9.1 (K), J4.1 (Pin_1), R18.2, RV3.1
- net V_shant: now reaches Q4.3 (S), R2.1, R6.1
- net V_ntc: now reaches J4.2 (Pin_2), R13.1, U1.10 (+)
- net at K1.2: now also D7.1 (K), R14.1
- net V_max_A: now reaches Q5.2 (G), RV2.2
- net V_Led_G: now reaches D12.2 (A), R19.2
- net V_op_T: now reaches R16.1, U1.8
- net V_out: now reaches J3.1 (Pin_1), R12.1, R19.1, R2.2, R7.1
- net V_Vmax-: now reaches R12.2, R20.1, U1.6 (-)
- net V_max_T: now reaches RV3.2, U1.9 (-)
- net V_Led_Red: now reaches D11.2 (A), R4.2
- net V_in renamed V_in-
- new net V_Vmax: C6.1, RV1.2, U1.5 (+)
Other:
- moved on the sheet: D12, R11, R16, R4, R6, R8
